File: auxi.kicad_pcb (KiCad board)
At the start: 2 copper layers, 110 x 140 mm, 49 parts

Commit message: Move the ESP32-CAM to the front (almost centered) and the sensors to its right
The camera is now at x = 146.5 (14.5 mm left of the board centre) and the
three sensor connectors sit to its right along the front edge. Camera
UART/5V lanes and the sensor lines were laid out by hand, the rest by
Freerouting. 167 tracks on one layer, DRC 0 errors, 0 unconnected; the PCB
nets still match the schematic pin by pin. README, CLAUDE.md, PDFs and
renders regenerated.

Co-Authored-By: Claude Sonnet 5.5 <noreply@anthropic.com>
Claude-Session: https://claude.ai/code/session_01V1Casvb8MJmuQffuKiRczF
Parts:
- moved J_LED_POWER1 26.2 mm to (204.0, 53.0)
- moved U_CAM1 25.5 mm to (135.1, 86.3)
- moved U_CAM2 25.5 mm to (157.9, 86.3)
- moved R1 25.3 mm to (208.0, 62.0), turned to 180 degrees
- moved C15 18.8 mm to (185.0, 75.5), turned to -90 degrees
- moved C1 17.5 mm to (198.0, 104.0), turned to 90 degrees
- moved C6 17.3 mm to (194.5, 118.0), turned to -90 degrees
- moved R2 14.7 mm to (178.5, 127.0), turned to 0 degrees
- moved J_SENSOR_FRONT1 14.0 mm to (175.0, 53.0)
- moved J_SENSOR_LEFT1 14.0 mm to (165.0, 53.0)
- moved J_SENSOR_RIGHT1 14.0 mm to (185.0, 53.0)
- moved C18 13.6 mm to (165.0, 75.5), turned to -90 degrees
- moved C16 13.3 mm to (175.0, 75.5), turned to -90 degrees
- moved C7 12.3 mm to (130.0, 148.0), turned to 0 degrees
- moved C17 11.3 mm to (170.5, 75.5), turned to -90 degrees
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Routing:
- net +VBAT_SW: track 252.5 -> 295.4 mm
- net GND: track 46.4 -> 8.50 mm
- net XSHUT_RIGHT: track 80.9 -> 110.4 mm
- net UART_ESP_TO_CAM: track 112.7 -> 87.2 mm
- net UART_CAM_TO_ESP: track 115.2 -> 89.7 mm
- net XSHUT_FRONT: track 80.0 -> 104.9 mm
- net +5V: track 153.0 -> 174.3 mm
- net STBY: track 10.6 -> 21.4 mm
- net SDA: track 125.2 -> 133.5 mm
- net LED_POWER_A: track 4.16 -> 10.8 mm
- net XSHUT_LEFT: track 93.9 -> 99.4 mm
- net +5V_ESP: track 15.0 -> 20.5 mm
- net SCL: track 129.4 -> 126.5 mm
- net +3V3: track 232.3 -> 231.2 mm
