File: auxi.kicad_pcb (KiCad board)
At the start: 2 copper layers, 110 x 140 mm, 49 parts

Commit message: Proximity LEDs soldered directly on the PCB; power LED is green
- The three 5 mm proximity LEDs go straight into the J_LED_* hole pairs
  (right hole / square pad = anode). No header or Dupont jumpers for them.
- Power LED is green (value, notes, BOM and docs updated; R1 1.5 kohm
  still valid: about 2.6 mA at 6.0 V and 4.2 mA at 8.4 V).
- No copper change: ERC 0, DRC 0 errors / 0 unconnected.
- README, CLAUDE.md, schematic notes, PDFs and BOM updated.

Co-Authored-By: Claude Sonnet 5.5 <noreply@anthropic.com>
Claude-Session: https://claude.ai/code/session_01V1Casvb8MJmuQffuKiRczF
Parts:
- J_LED_POWER1: value POWER LED (azul) -> POWER LED (verde)
Changed lines of the file:
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@@
 			)
 		)
-		(property "Value" "POWER LED (azul)"
+		(property "Value" "POWER LED (verde)"
 			(at 0 4.92 0)
 			(layer "F.Fab")

Commit message: C3 (motor supply) is 220 uF 16 V instead of 25 V
The rail is 8.4 V at most, so a 16 V part keeps a wide margin.

Co-Authored-By: Claude Sonnet 5.5 <noreply@anthropic.com>
Claude-Session: https://claude.ai/code/session_01V1Casvb8MJmuQffuKiRczF
Parts:
- C3: value 220uF 25V -> 220uF 16V
Changed lines of the file:
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@@
 			)
 		)
-		(property "Value" "220uF 25V"
+		(property "Value" "220uF 16V"
 			(at 1.75 5.25 0)
 			(layer "F.Fab")

Commit message: Chassis v8 update: LEDs soldered on the PCB, battery on a screw terminal
PCB copper, footprints and tracks are unchanged. Updated the 3D models
(colored 5 mm LEDs in auxi.3dshapes/, screw terminal for J_BAT1), the
schematic descriptions and notes, CLAUDE.md and README.md.

Work in progress: ERC/DRC and the regeneration of docs/*.pdf and *.png
are still pending because kicad-cli was not available.

Co-Authored-By: Claude Sonnet 5.5 <noreply@anthropic.com>
Claude-Session: https://claude.ai/code/session_01HrZukSfyeMd8Be9PGS4Uge
Parts:
- J_BAT1: value XT30 BAT 2S -> BAT 2S (bornera)
Changed lines of the file:
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@@
 			)
 		)
-		(property "Value" "XT30 BAT 2S"
+		(property "Value" "BAT 2S (bornera)"
 			(at 2.5 4 0)
 			(layer "F.Fab")
@@
 		)
 		(embedded_fonts no)
-		(model "${KICAD10_3DMODEL_DIR}/Connector_AMASS.3dshapes/AMASS_XT30UPB-M_1x02_P5.0mm_Vertical.step"
+		(model "${KICAD10_3DMODEL_DIR}/TerminalBlock_Phoenix.3dshapes/TerminalBlock_Phoenix_MKDS-1,5-2-5.08_1x02_P5.08mm_Horizontal.step"
 			(offset
-				(xyz 0 0 0)
+				(xyz -0.04 0 0)
 			)
 			(scale
@@
 		)
 		(embedded_fonts no)
-		(model "${KICAD10_3DMODEL_DIR}/Connector_PinHeader_2.54mm.3dshapes/PinHeader_1x02_P2.54mm_Vertical.step"
+		(model "${KIPRJMOD}/auxi.3dshapes/LED_D5.0mm_Green.wrl"
 			(offset
-				(xyz 0 0 0)
+				(xyz 0 -1.27 0)
 			)
 			(scale
@@
 		)
 		(embedded_fonts no)
-		(model "${KICAD10_3DMODEL_DIR}/Connector_PinHeader_2.54mm.3dshapes/PinHeader_1x02_P2.54mm_Vertical.step"
+		(model "${KIPRJMOD}/auxi.3dshapes/LED_D5.0mm_Green.wrl"
 			(offset
-				(xyz 0 0 0)
+				(xyz 0 -1.27 0)
 			)
 			(scale
@@
 		)
 		(embedded_fonts no)
-		(model "${KICAD10_3DMODEL_DIR}/Connector_PinHeader_2.54mm.3dshapes/PinHeader_1x02_P2.54mm_Vertical.step"
+		(model "${KIPRJMOD}/auxi.3dshapes/LED_D5.0mm_Yellow.wrl"
 			(offset
-				(xyz 0 0 0)
+				(xyz 0 -1.27 0)
 			)
 			(scale
@@
 		)
 		(embedded_fonts no)
-		(model "${KICAD10_3DMODEL_DIR}/Connector_PinHeader_2.54mm.3dshapes/PinHeader_1x02_P2.54mm_Vertical.step"
+		(model "${KIPRJMOD}/auxi.3dshapes/LED_D5.0mm_Red.wrl"
 			(offset
-				(xyz 0 0 0)
+				(xyz 0 -1.27 0)
 			)
 			(scale

Commit message: KiCad: SDA=GPIO7 y SCL=GPIO15 segun el firmware
Se renombran las redes SDA/SCL sin mover pistas. En los conectores de
sensor el orden pasa a 3=SCL, 4=SDA.

Co-Authored-By: Claude Sonnet 5.5 <noreply@anthropic.com>
Connections:
- J_SENSOR_FRONT1 pad 3: SDA -> SCL
- J_SENSOR_FRONT1 pad 4: SCL -> SDA
- J_SENSOR_LEFT1 pad 3: SDA -> SCL
- J_SENSOR_LEFT1 pad 4: SCL -> SDA
- J_SENSOR_RIGHT1 pad 3: SDA -> SCL
- J_SENSOR_RIGHT1 pad 4: SCL -> SDA
- U_ESP_J1 pad 7: SCL -> SDA
- U_ESP_J1 pad 8: SDA -> SCL
Routing:
- net SDA: track 133.5 -> 126.5 mm
- net SCL: track 126.5 -> 133.5 mm
Other:
- board text added: "JST: 1=3V3 2=GND 3=SCL 4=SDA 5=XSHUT"
- board text removed: "JST: 1=3V3 2=GND 3=SDA 4=SCL 5=XSHUT"
Changed lines of the file:
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@@
 			(layers "*.Cu" "*.Mask")
 			(remove_unused_layers no)
-			(net "SDA")
+			(net "SCL")
 		)
 		(pad "4" thru_hole oval
@@
 			(layers "*.Cu" "*.Mask")
 			(remove_unused_layers no)
-			(net "SCL")
+			(net "SDA")
 		)
 		(pad "5" thru_hole oval
@@
 			(layers "*.Cu" "*.Mask")
 			(remove_unused_layers no)
-			(net "SDA")
+			(net "SCL")
 		)
 		(pad "4" thru_hole oval
@@
 			(layers "*.Cu" "*.Mask")
 			(remove_unused_layers no)
-			(net "SCL")
+			(net "SDA")
 		)
 		(pad "5" thru_hole oval
@@
 			(layers "*.Cu" "*.Mask")
 			(remove_unused_layers no)
-			(net "SDA")
+			(net "SCL")
 		)
 		(pad "4" thru_hole oval
@@
 			(layers "*.Cu" "*.Mask")
 			(remove_unused_layers no)
-			(net "SCL")
+			(net "SDA")
 		)
 		(pad "5" thru_hole oval
@@
 			(layers "*.Cu" "*.Mask")
 			(remove_unused_layers no)
-			(net "SCL")
+			(net "SDA")
 		)
 		(pad "8" thru_hole circle
@@
 			(layers "*.Cu" "*.Mask")
 			(remove_unused_layers no)
-			(net "SDA")
+			(net "SCL")
 		)
 		(pad "9" thru_hole circle
@@
 		)
 	)
-	(gr_text "JST: 1=3V3 2=GND 3=SDA 4=SCL 5=XSHUT"
+	(gr_text "JST: 1=3V3 2=GND 3=SCL 4=SDA 5=XSHUT"
 		(at 172 108 0)
 		(layer "F.SilkS")
@@
 		(width 0.4)
 		(layer "B.Cu")
-		(net "SDA")
+		(net "SCL")
 	)
 	(segment
@@
 		(width 0.4)
 		(layer "B.Cu")
-		(net "SDA")
+		(net "SCL")
 	)
 	(segment
@@
 		(width 0.4)
 		(layer "B.Cu")
-		(net "SDA")
+		(net "SCL")
 	)
 	(segment
@@
 		(width 0.4)
 		(layer "B.Cu")
-		(net "SDA")
+		(net "SCL")
 	)
 	(segment
@@
 		(width 0.4)
 		(layer "B.Cu")
-		(net "SDA")
+		(net "SCL")
 	)
 	(segment
@@
 		(width 0.4)
 		(layer "B.Cu")
-		(net "SDA")
+		(net "SCL")
 	)
 	(segment
@@
 		(width 0.4)
 		(layer "B.Cu")
-		(net "SDA")
+		(net "SCL")
 	)
 	(segment
@@
 		(width 0.4)
 		(layer "B.Cu")
-		(net "SCL")
+		(net "SDA")
 	)
 	(segment
@@
 		(width 0.4)
 		(layer "B.Cu")
-		(net "SCL")
+		(net "SDA")
 	)
 	(segment
@@
 		(width 0.4)
 		(layer "B.Cu")
-		(net "SCL")
+		(net "SDA")
 	)
 	(segment
@@
 		(width 0.4)
 		(layer "B.Cu")
-		(net "SCL")
+		(net "SDA")
 	)
 	(segment
@@
 		(width 0.4)
 		(layer "B.Cu")
-		(net "SCL")
+		(net "SDA")
 	)
 	(segment
@@
 		(width 0.4)
 		(layer "B.Cu")
-		(net "SCL")
+		(net "SDA")
 	)
 	(segment
@@
 		(width 0.4)
 		(layer "B.Cu")
-		(net "SCL")
+		(net "SDA")
 	)
 	(segment
