File: auxi.kicad_sch (KiCad schematic)
At the start: 45 parts

Commit message: Proximity LEDs soldered directly on the PCB; power LED is green
- The three 5 mm proximity LEDs go straight into the J_LED_* hole pairs
  (right hole / square pad = anode). No header or Dupont jumpers for them.
- Power LED is green (value, notes, BOM and docs updated; R1 1.5 kohm
  still valid: about 2.6 mA at 6.0 V and 4.2 mA at 8.4 V).
- No copper change: ERC 0, DRC 0 errors / 0 unconnected.
- README, CLAUDE.md, schematic notes, PDFs and BOM updated.

Co-Authored-By: Claude Sonnet 5.5 <noreply@anthropic.com>
Claude-Session: https://claude.ai/code/session_01V1Casvb8MJmuQffuKiRczF
Parts:
- J_LED_POWER1: value POWER LED (azul) -> POWER LED (verde)
Other:
- note added: "6. LEDs DE PROXIMIDAD (reglamento, soldados en la placa)"
- note added: "FRONT = ROJO, LEFT = AMARILLO, RIGHT = VERDE. Encendido si distancia <= 100 mm. Los LED de 5 mm se sueldan DIRECTO en los pares de agujeros J_LED_* (pata larga = anodo = pad cuadrado, junto a la resistencia). Pin 1 = LED+ (anodo), pin 2 = LED- (GND). ~2.5-3 mA a 3.3 V. R5 (verde) PROVISIONAL: 470 ohm vale para verde clasico (Vf ~2.1 V); hay que recalcularla si el LED es verde brillante (Vf ~3 V)."
- note added: "J_BAT1 (XT30UPB-M): pin 1 = BAT- (lado biselado), pin 2 = BAT+ (lado plano). J_SWITCH1: interruptor externo. Por aqui pasa TODA la corriente del robot: bornera 5.08 mm y cable 20 AWG, nunca Dupont. R1 1.5k: LED verde de funcionamiento, ~2.6 mA (6.0 V) - ~4.2 mA (8.4 V). Calibrar el MP1584 a 5.0 V con multimetro ANTES de enchufar cualquier modulo. D1 (Schottky): evita que el USB del PC alimente el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"
- note removed: "6. LEDs DE PROXIMIDAD (reglamento, externos)"
- note removed: "FRONT = ROJO, LEFT = AMARILLO, RIGHT = VERDE. Encendido si distancia <= 100 mm. Pin 1 = LED+ (anodo), pin 2 = LED- (GND). ~2.5-3 mA a 3.3 V. R7 (verde) PROVISIONAL: 470 ohm vale para verde clasico (Vf ~2.1 V); hay que recalcularla si el LED es verde brillante (Vf ~3 V)."
- note removed: "J_BAT1 (XT30UPB-M): pin 1 = BAT- (lado biselado), pin 2 = BAT+ (lado plano). J_SWITCH1: interruptor externo. Por aqui pasa TODA la corriente del robot: bornera 5.08 mm y cable 20 AWG, nunca Dupont. R1 1.5k: LED azul a 2.0 mA (6.0 V) - 3.6 mA (8.4 V). Calibrar el MP1584 a 5.0 V con multimetro ANTES de enchufar cualquier modulo. D1 (Schottky): evita que el USB del PC alimente el robot y viceversa. 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"
Changed lines of the file:
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@@
 		)
 	)
-	(text "J_BAT1 (XT30UPB-M): pin 1 = BAT- (lado biselado), pin 2 = BAT+ (lado plano).\nJ_SWITCH1: interruptor externo. Por aqui pasa TODA la corriente del robot:\nbornera 5.08 mm y cable 20 AWG, nunca Dupont.\nR1 1.5k: LED azul a 2.0 mA (6.0 V) - 3.6 mA (8.4 V).\nCalibrar el MP1584 a 5.0 V con multimetro ANTES de enchufar cualquier modulo.\nD1 (Schottky): evita que el USB del PC alimente el robot y viceversa.\nPWR_FLAG: +VBAT_SW, GND y +5V_ESP solo reciben corriente a traves de\nconectores o del diodo (pines pasivos); las banderas le indican al ERC\nque esas redes SI estan alimentadas."
+	(text "J_BAT1 (XT30UPB-M): pin 1 = BAT- (lado biselado), pin 2 = BAT+ (lado plano).\nJ_SWITCH1: interruptor externo. Por aqui pasa TODA la corriente del robot:\nbornera 5.08 mm y cable 20 AWG, nunca Dupont.\nR1 1.5k: LED verde de funcionamiento, ~2.6 mA (6.0 V) - ~4.2 mA (8.4 V).\nCalibrar el MP1584 a 5.0 V con multimetro ANTES de enchufar cualquier modulo.\nD1 (Schottky): evita que el USB del PC alimente el robot y viceversa.\nPWR_FLAG: +VBAT_SW, GND y +5V_ESP solo reciben corriente a traves de\nconectores o del diodo (pines pasivos); las banderas le indican al ERC\nque esas redes SI estan alimentadas."
 		(exclude_from_sim no)
 		(at 20 320 0)
@@
 		)
 	)
-	(text "6. LEDs DE PROXIMIDAD (reglamento, externos)"
+	(text "6. LEDs DE PROXIMIDAD (reglamento, soldados en la placa)"
 		(exclude_from_sim no)
 		(at 150 203 0)
@@
 		)
 	)
-	(text "FRONT = ROJO, LEFT = AMARILLO, RIGHT = VERDE. Encendido si distancia <= 100 mm.\nPin 1 = LED+ (anodo), pin 2 = LED- (GND). ~2.5-3 mA a 3.3 V.\nR7 (verde) PROVISIONAL: 470 ohm vale para verde clasico (Vf ~2.1 V);\nhay que recalcularla si el LED es verde brillante (Vf ~3 V)."
+	(text "FRONT = ROJO, LEFT = AMARILLO, RIGHT = VERDE. Encendido si distancia <= 100 mm.\nLos LED de 5 mm se sueldan DIRECTO en los pares de agujeros J_LED_*\n(pata larga = anodo = pad cuadrado, junto a la resistencia).\nPin 1 = LED+ (anodo), pin 2 = LED- (GND). ~2.5-3 mA a 3.3 V.\nR5 (verde) PROVISIONAL: 470 ohm vale para verde clasico (Vf ~2.1 V);\nhay que recalcularla si el LED es verde brillante (Vf ~3 V)."
 		(exclude_from_sim no)
 		(at 150 222 0)
@@
 			)
 		)
-		(property "Value" "POWER LED (azul)"
+		(property "Value" "POWER LED (verde)"
 			(at 92.71 288.29 0)
 			(effects

Commit message: C3 (motor supply) is 220 uF 16 V instead of 25 V
The rail is 8.4 V at most, so a 16 V part keeps a wide margin.

Co-Authored-By: Claude Sonnet 5.5 <noreply@anthropic.com>
Claude-Session: https://claude.ai/code/session_01V1Casvb8MJmuQffuKiRczF
Parts:
- C3: value 220uF 25V -> 220uF 16V
Changed lines of the file:
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@@
 			)
 		)
-		(property "Value" "220uF 25V"
+		(property "Value" "220uF 16V"
 			(at 381.0 148.59 0)
 			(effects

Commit message: Chassis v8 update: LEDs soldered on the PCB, battery on a screw terminal
PCB copper, footprints and tracks are unchanged. Updated the 3D models
(colored 5 mm LEDs in auxi.3dshapes/, screw terminal for J_BAT1), the
schematic descriptions and notes, CLAUDE.md and README.md.

Work in progress: ERC/DRC and the regeneration of docs/*.pdf and *.png
are still pending because kicad-cli was not available.

Co-Authored-By: Claude Sonnet 5.5 <noreply@anthropic.com>
Claude-Session: https://claude.ai/code/session_01HrZukSfyeMd8Be9PGS4Uge
Parts:
- J_BAT1: value XT30 BAT 2S -> BAT 2S (bornera)
Other:
- note added: "J_BAT1 = bornera 5.08 mm en los pads del XT30UPB-M: pin 1 = BAT- ('-'), pin 2 = BAT+ ('+'). J_SWITCH1: interruptor externo. Por aqui pasa TODA la corriente del robot: bornera 5.08 mm y cable 20 AWG, nunca Dupont (igual que la bateria). R1 1.5k: LED verde soldado directo en J_LED_POWER1, ~2.6 mA (6.0 V) - ~4.2 mA (8.4 V). Calibrar el MP1584 a 5.0 V con multimetro ANTES de enchufar cualquier modulo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"
- note removed: "J_BAT1 (XT30UPB-M): pin 1 = BAT- (lado biselado), pin 2 = BAT+ (lado plano). J_SWITCH1: interruptor externo. Por aqui pasa TODA la corriente del robot: bornera 5.08 mm y cable 20 AWG, nunca Dupont. R1 1.5k: LED verde de funcionamiento, ~2.6 mA (6.0 V) - ~4.2 mA (8.4 V). Calibrar el MP1584 a 5.0 V con multimetro ANTES de enchufar cualquier modulo. D1 (Schottky): evita que el USB del PC alimente el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"
Changed lines of the file:
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@@
 		)
 	)
-	(text "J_BAT1 (XT30UPB-M): pin 1 = BAT- (lado biselado), pin 2 = BAT+ (lado plano).\nJ_SWITCH1: interruptor externo. Por aqui pasa TODA la corriente del robot:\nbornera 5.08 mm y cable 20 AWG, nunca Dupont.\nR1 1.5k: LED verde de funcionamiento, ~2.6 mA (6.0 V) - ~4.2 mA (8.4 V).\nCalibrar el MP1584 a 5.0 V con multimetro ANTES de enchufar cualquier modulo.\nD1 (Schottky): evita que el USB del PC alimente el robot y viceversa.\nPWR_FLAG: +VBAT_SW, GND y +5V_ESP solo reciben corriente a traves de\nconectores o del diodo (pines pasivos); las banderas le indican al ERC\nque esas redes SI estan alimentadas."
+	(text "J_BAT1 = bornera 5.08 mm en los pads del XT30UPB-M: pin 1 = BAT- ('-'), pin 2 = BAT+ ('+').\nJ_SWITCH1: interruptor externo. Por aqui pasa TODA la corriente del robot:\nbornera 5.08 mm y cable 20 AWG, nunca Dupont (igual que la bateria).\nR1 1.5k: LED verde soldado directo en J_LED_POWER1, ~2.6 mA (6.0 V) - ~4.2 mA (8.4 V).\nCalibrar el MP1584 a 5.0 V con multimetro ANTES de enchufar cualquier modulo.\nD1 (Schottky): evita que el USB del PC alimente el robot y viceversa.\nPWR_FLAG: +VBAT_SW, GND y +5V_ESP solo reciben corriente a traves de\nconectores o del diodo (pines pasivos); las banderas le indican al ERC\nque esas redes SI estan alimentadas."
 		(exclude_from_sim no)
 		(at 20 320 0)
@@
 			)
 		)
-		(property "Description" "Header macho 1x2 (2.54 mm) para LED externo con jumpers Dupont. Pin 1 = LED+ (anodo), pin 2 = LED- (catodo/GND)."
+		(property "Description" "Par de agujeros 1x2 (2.54 mm) para un LED de 5 mm soldado directamente en la placa (sin header ni Dupont). Pin 1 = LED+ (anodo, pata larga, pad cuadrado), pin 2 = LED- (catodo/GND)."
 			(at 187.96 154.94 0)
 			(hide yes)
@@
 			)
 		)
-		(property "Description" "Header macho 1x2 (2.54 mm) para LED externo con jumpers Dupont. Pin 1 = LED+ (anodo), pin 2 = LED- (catodo/GND)."
+		(property "Description" "Par de agujeros 1x2 (2.54 mm) para un LED de 5 mm soldado directamente en la placa (sin header ni Dupont). Pin 1 = LED+ (anodo, pata larga, pad cuadrado), pin 2 = LED- (catodo/GND)."
 			(at 187.96 170.18 0)
 			(hide yes)
@@
 			)
 		)
-		(property "Description" "Header macho 1x2 (2.54 mm) para LED externo con jumpers Dupont. Pin 1 = LED+ (anodo), pin 2 = LED- (catodo/GND)."
+		(property "Description" "Par de agujeros 1x2 (2.54 mm) para un LED de 5 mm soldado directamente en la placa (sin header ni Dupont). Pin 1 = LED+ (anodo, pata larga, pad cuadrado), pin 2 = LED- (catodo/GND)."
 			(at 187.96 185.42 0)
 			(hide yes)
@@
 			)
 		)
-		(property "Value" "XT30 BAT 2S"
+		(property "Value" "BAT 2S (bornera)"
 			(at 29.21 255.27 0)
 			(effects
@@
 			)
 		)
-		(property "Description" "Header macho 1x2 (2.54 mm) para LED externo con jumpers Dupont. Pin 1 = LED+ (anodo), pin 2 = LED- (catodo/GND)."
+		(property "Description" "Par de agujeros 1x2 (2.54 mm) para un LED de 5 mm soldado directamente en la placa (sin header ni Dupont). Pin 1 = LED+ (anodo, pata larga, pad cuadrado), pin 2 = LED- (catodo/GND)."
 			(at 106.68 284.48 0)
 			(hide yes)
